Commit message: added rc_visard to cob_bringup

File: cob_hardware_config/robots/cob4-7/urdf/calibration_default.urdf.xacro (robot description, xacro)
@@ -102,10 +102,10 @@
 	<xacro:property name="def_torso_cam3d_down_yaw" value="0.0"/>
 	<!-- sensorring cam3d mount positions | relative to sensorring_link -->
-	<xacro:property name="def_sensorring_cam3d_x" value="0.1251"/>
-	<xacro:property name="def_sensorring_cam3d_y" value="0.0"/>
-	<xacro:property name="def_sensorring_cam3d_z" value="0.001"/>
-	<xacro:property name="def_sensorring_cam3d_roll" value="0.0"/>
+	<xacro:property name="def_sensorring_cam3d_x" value="0.122"/>
+	<xacro:property name="def_sensorring_cam3d_y" value="0.081"/>
+	<xacro:property name="def_sensorring_cam3d_z" value="0.040"/>
+	<xacro:property name="def_sensorring_cam3d_roll" value="-1.57079"/>
 	<xacro:property name="def_sensorring_cam3d_pitch" value="0.0"/>
-	<xacro:property name="def_sensorring_cam3d_yaw" value="0.0"/>
+	<xacro:property name="def_sensorring_cam3d_yaw" value="-1.57079"/>
 	<!-- head cam mount positions | relative to head_3_link -->
 	<xacro:property name="def_head_cam_x" value="-0.181"/>

File: cob_hardware_config/robots/cob4-7/urdf/cob4-7.urdf.xacro (robot description, xacro)
@@ -23,4 +23,5 @@
   <xacro:include filename="$(find cob_description)/urdf/sensors/realsense_zr300.urdf.xacro" />
   <xacro:include filename="$(find cob_description)/urdf/sensors/kinect.urdf.xacro" />
+  <xacro:include filename="$(find cob_description)/urdf/sensors/rc_visard160.urdf.xacro" />
   <xacro:include filename="$(find cob_description)/urdf/sensors/usb_cam.urdf.xacro" />
   <xacro:include filename="$(find cob_description)/urdf/sensors/sick_s300_laser.urdf.xacro"/>
@@ -67,7 +68,10 @@
     <origin xyz="${sensorring_x} ${sensorring_y} ${sensorring_z}" rpy="${sensorring_roll} ${sensorring_pitch} ${sensorring_yaw}" />
   </xacro:sensorring>
-  <xacro:cob_kinect_v0 name="sensorring_cam3d" ros_topic="sensorring_cam3d" parent="sensorring_link" update_rate="30" data_skip="9">
+  <xacro:rc_160 name="sensorring_cam3d" ros_topic="sensorring_cam3d" parent="sensorring_link" update_rate="30" data_skip="9">
     <origin xyz="${sensorring_cam3d_x} ${sensorring_cam3d_y} ${sensorring_cam3d_z}" rpy="${sensorring_cam3d_roll} ${sensorring_cam3d_pitch} ${sensorring_cam3d_yaw}" />
-  </xacro:cob_kinect_v0>
+  </xacro:rc_160>
+  <!--xacro:cob_kinect_v0 name="sensorring_cam3d" ros_topic="sensorring_cam3d" parent="sensorring_link" update_rate="30" data_skip="9">
+    <origin xyz="${sensorring_cam3d_x} ${sensorring_cam3d_y} ${sensorring_cam3d_z}" rpy="${sensorring_cam3d_roll} ${sensorring_cam3d_pitch} ${sensorring_cam3d_yaw}" />
+  </xacro:cob_kinect_v0-->
   <!-- grippers -->
   <xacro:gripper name="gripper_right" parent="arm_right_7_link">

Commit message: added PTP start for rc_visard

File: cob_hardware_config/robots/cob4-7/urdf/calibration_default.urdf.xacro (robot description, xacro)
@@ -102,10 +102,13 @@
 	<xacro:property name="def_torso_cam3d_down_yaw" value="0.0"/>
 	<!-- sensorring cam3d mount positions | relative to sensorring_link -->
-	<xacro:property name="def_sensorring_cam3d_x" value="0.122"/>
+	<!--xacro:property name="def_sensorring_cam3d_x" value="0.122"/>
 	<xacro:property name="def_sensorring_cam3d_y" value="0.081"/>
-	<xacro:property name="def_sensorring_cam3d_z" value="0.040"/>
-	<xacro:property name="def_sensorring_cam3d_roll" value="-1.57079"/>
-	<xacro:property name="def_sensorring_cam3d_pitch" value="0.0"/>
-	<xacro:property name="def_sensorring_cam3d_yaw" value="-1.57079"/>
+	<xacro:property name="def_sensorring_cam3d_z" value="0.040"/-->
+	<xacro:property name="def_sensorring_cam3d_x" value="0.11375"/>
+	<xacro:property name="def_sensorring_cam3d_y" value="0.0812894"/>
+	<xacro:property name="def_sensorring_cam3d_z" value="0.0129219"/>
+	<xacro:property name="def_sensorring_cam3d_roll" value="-1.56955"/>
+	<xacro:property name="def_sensorring_cam3d_pitch" value="0.00965916"/>
+	<xacro:property name="def_sensorring_cam3d_yaw" value="-1.60063"/>
 	<!-- head cam mount positions | relative to head_3_link -->
 	<xacro:property name="def_head_cam_x" value="-0.181"/>
