Commit message: added cob4-25 robot

File: cob_hardware_config/robots/cob4-25/urdf/calibration_default.urdf.xacro (robot description, xacro)
@@ -49,4 +49,32 @@
 	<xacro:property name="def_sensorring_pitch" value="0.0"/>
 	<xacro:property name="def_sensorring_yaw" value="0.0"/>
+	<!-- arm right mount positions | relative to torso_3_link -->
+	<xacro:property name="def_arm_right_x" value="0.0"/>
+	<xacro:property name="def_arm_right_y" value="-0.014"/>
+	<xacro:property name="def_arm_right_z" value="0.55"/>
+	<xacro:property name="def_arm_right_roll" value="1.57097"/>
+	<xacro:property name="def_arm_right_pitch" value="0"/>
+	<xacro:property name="def_arm_right_yaw" value="0.0"/>
+	<!-- arm left mount positions | relative to torso_3_link -->
+	<xacro:property name="def_arm_left_x" value="0.0"/>
+	<xacro:property name="def_arm_left_y" value="0.014"/>
+	<xacro:property name="def_arm_left_z" value="0.55"/>
+	<xacro:property name="def_arm_left_roll" value="1.57097"/>
+	<xacro:property name="def_arm_left_pitch" value="0"/>
+	<xacro:property name="def_arm_left_yaw" value="3.14159"/>
+	<!-- gripper right mount positions | relative to arm_right_7_link -->
+	<xacro:property name="def_gripper_right_x" value="0.0"/>
+	<xacro:property name="def_gripper_right_y" value="0.0"/>
+	<xacro:property name="def_gripper_right_z" value="0.0748"/>
+	<xacro:property name="def_gripper_right_roll" value="0.0"/>
+	<xacro:property name="def_gripper_right_pitch" value="0.0"/>
+	<xacro:property name="def_gripper_right_yaw" value="3.14159"/>
+	<!-- gripper left mount positions | relative to arm_left_7_link -->
+	<xacro:property name="def_gripper_left_x" value="0.0"/>
+	<xacro:property name="def_gripper_left_y" value="0.0"/>
+	<xacro:property name="def_gripper_left_z" value="0.0748"/>
+	<xacro:property name="def_gripper_left_roll" value="0.0"/>
+	<xacro:property name="def_gripper_left_pitch" value="0.0"/>
+	<xacro:property name="def_gripper_left_yaw" value="3.14159"/>
 	<!-- ***************************** -->
 	<!-- extrinsic camera calibration  -->
@@ -74,10 +102,13 @@
 	<xacro:property name="def_torso_cam3d_down_yaw" value="0.0"/>
 	<!-- sensorring cam3d mount positions | relative to sensorring_link -->
-	<xacro:property name="def_sensorring_cam3d_x" value="0.1251"/>
-	<xacro:property name="def_sensorring_cam3d_y" value="0.0"/>
-	<xacro:property name="def_sensorring_cam3d_z" value="0.001"/>
-	<xacro:property name="def_sensorring_cam3d_roll" value="0.0"/>
-	<xacro:property name="def_sensorring_cam3d_pitch" value="0.0"/>
-	<xacro:property name="def_sensorring_cam3d_yaw" value="0.0"/>
+	<!--xacro:property name="def_sensorring_cam3d_x" value="0.122"/>
+	<xacro:property name="def_sensorring_cam3d_y" value="0.081"/>
+	<xacro:property name="def_sensorring_cam3d_z" value="0.040"/-->
+	<xacro:property name="def_sensorring_cam3d_x" value="0.11375"/>
+	<xacro:property name="def_sensorring_cam3d_y" value="0.0812894"/>
+	<xacro:property name="def_sensorring_cam3d_z" value="0.0129219"/>
+	<xacro:property name="def_sensorring_cam3d_roll" value="-1.56955"/>
+	<xacro:property name="def_sensorring_cam3d_pitch" value="0.00965916"/>
+	<xacro:property name="def_sensorring_cam3d_yaw" value="-1.60063"/>
 	<!-- head cam mount positions | relative to head_3_link -->
 	<xacro:property name="def_head_cam_x" value="-0.181"/>

File: cob_hardware_config/robots/cob4-25/urdf/cob4-25.urdf.xacro (robot description, xacro)
@@ -11,4 +11,8 @@
   <!-- torso -->
   <xacro:include filename="$(find cob_description)/urdf/cob4_torso/torso.urdf.xacro" />
+  <!-- arm -->
+  <xacro:include filename="$(find cob_description)/urdf/cob4_arm/cob4_arm.urdf.xacro" />
+  <!-- hand -->
+  <xacro:include filename="$(find cob_description)/urdf/cob4_gripper/gripper.urdf.xacro" />
   <!-- head -->
   <xacro:include filename="$(find cob_description)/urdf/cob4_head/head.urdf.xacro" />
@@ -19,4 +23,5 @@
   <xacro:include filename="$(find cob_description)/urdf/sensors/usb_cam.urdf.xacro" />
   <xacro:include filename="$(find cob_description)/urdf/sensors/sick_s300_laser.urdf.xacro"/>
+  <xacro:include filename="$(find cob_description)/urdf/sensors/rc_visard160.urdf.xacro" />
   <!-- composition of the robot -->
   <xacro:base name="base"/>
@@ -49,9 +54,25 @@
     <origin xyz="${head_cam_x} ${head_cam_y} ${head_cam_z}" rpy="${head_cam_roll} ${head_cam_pitch} ${head_cam_yaw}" />
   </xacro:usb_cam>
+  <xacro:cob4_arm name="arm_right" parent="torso_3_link" has_podest="false">
+    <origin xyz="${arm_right_x} ${arm_right_y} ${arm_right_z}" rpy="${arm_right_roll} ${arm_right_pitch} ${arm_right_yaw}" />
+  </xacro:cob4_arm>
+  <xacro:cob4_arm name="arm_left" parent="torso_3_link" has_podest="false">
+    <origin xyz="${arm_left_x} ${arm_left_y} ${arm_left_z}" rpy="${arm_left_roll} ${arm_left_pitch} ${arm_left_yaw}" />
+  </xacro:cob4_arm>
   <xacro:sensorring name="sensorring" parent="head_3_link" active="false">
     <origin xyz="${sensorring_x} ${sensorring_y} ${sensorring_z}" rpy="${sensorring_roll} ${sensorring_pitch} ${sensorring_yaw}" />
   </xacro:sensorring>
-  <xacro:realsense_d435 name="sensorring_cam3d" parent="sensorring_link">
+  <xacro:rc_160 prefix="sensorring_cam3d_" parent="sensorring_link">
     <origin xyz="${sensorring_cam3d_x} ${sensorring_cam3d_y} ${sensorring_cam3d_z}" rpy="${sensorring_cam3d_roll} ${sensorring_cam3d_pitch} ${sensorring_cam3d_yaw}" />
-  </xacro:realsense_d435>
+  </xacro:rc_160>
+  <!--xacro:realsense_d435 name="sensorring_cam3d" parent="sensorring_link">
+    <origin xyz="${sensorring_cam3d_x} ${sensorring_cam3d_y} ${sensorring_cam3d_z}" rpy="${sensorring_cam3d_roll} ${sensorring_cam3d_pitch} ${sensorring_cam3d_yaw}" />
+  </xacro:realsense_d435-->
+  <!-- grippers -->
+  <xacro:gripper name="gripper_right" parent="arm_right_7_link">
+    <origin xyz="${gripper_right_x} ${gripper_right_y} ${gripper_right_z}" rpy="${gripper_right_roll} ${gripper_right_pitch} ${gripper_right_yaw}" />
+  </xacro:gripper>
+  <xacro:gripper name="gripper_left" parent="arm_left_7_link">
+    <origin xyz="${gripper_left_x} ${gripper_left_y} ${gripper_left_z}" rpy="${gripper_left_roll} ${gripper_left_pitch} ${gripper_left_yaw}" />
+  </xacro:gripper>
 </robot>

File: cob_hardware_config/robots/cob4-25/urdf/properties.urdf.xacro (robot description, xacro)
@@ -66,4 +66,18 @@
 	<xacro:property name="arm_left_pitch" value="${def_arm_left_pitch+offset_arm_left_pitch}"/>
 	<xacro:property name="arm_left_yaw" value="${def_arm_left_yaw+offset_arm_left_yaw}"/>
+	<!-- gripper mount positions | relative to arm_7_link -->
+	<xacro:property name="gripper_right_x" value="${def_gripper_right_x+offset_gripper_right_x}"/>
+	<xacro:property name="gripper_right_y" value="${def_gripper_right_y+offset_gripper_right_y}"/>
+	<xacro:property name="gripper_right_z" value="${def_gripper_right_z+offset_gripper_right_z}"/>
+	<xacro:property name="gripper_right_roll" value="${def_gripper_right_roll+offset_gripper_right_roll}"/>
+	<xacro:property name="gripper_right_pitch" value="${def_gripper_right_pitch+offset_gripper_right_pitch}"/>
+	<xacro:property name="gripper_right_yaw" value="${def_gripper_right_yaw+offset_gripper_right_yaw}"/>
+	<!-- gripper mount positions | relative to arm_7_link -->
+	<xacro:property name="gripper_left_x" value="${def_gripper_left_x+offset_gripper_left_x}"/>
+	<xacro:property name="gripper_left_y" value="${def_gripper_left_y+offset_gripper_left_y}"/>
+	<xacro:property name="gripper_left_z" value="${def_gripper_left_z+offset_gripper_left_z}"/>
+	<xacro:property name="gripper_left_roll" value="${def_gripper_left_roll+offset_gripper_left_roll}"/>
+	<xacro:property name="gripper_left_pitch" value="${def_gripper_left_pitch+offset_gripper_left_pitch}"/>
+	<xacro:property name="gripper_left_yaw" value="${def_gripper_left_yaw+offset_gripper_left_yaw}"/>
 	<!-- *********************************** -->
 	<!-- kinematic chain reference positions -->
